File: zaza-motor-controller.sch (KiCad schematic (older format))
At the start: 85 parts, among them J1 VIN, J2 VIN, J200 MX120G, J3 CONN_02X05, J4 CONN_02X01, J5 U, J6 V, J7 CAL_EN, J8 CONN_01X06, Q1 NZT605, U1 74HC00, U10 LM7805CT, U100 IRS2003, U200 IRS2003, U3 LM358, U4 LM555N, U5 74xx138, U6 74xx595, U8 AT25XX, U9 ADS1018

Commit message: schematic moar cool scheise
Parts:
- removed J3: CONN_02X05, Connectors_Multicomp:Multicomp_MC9A12-1034_2x05x2.54mm_Straight, symbol CONN_02X05
- D1: footprint Diodes_THT:D_DO-35_SOD27_P7.62mm_Horizontal -> Diodes_SMD:D_MiniMELF_Standard
- D103, D203, D6: footprint Diodes_SMD:D_SOD-323 -> Diodes_SMD:D_SMA_Standard
- J200: footprint (none) -> molex-120g:Molex_MX120G_02x06_3.5mm_36783-1201
- QA1, QB1, QC1, QD1: footprint TO_SOT_Packages_SMD:SOT-404 -> TO-SMD:SOT-404-thermal-vias
Connections:
- net A: now also U1.13; no longer U1.2
- net C: now also U1.2; no longer U1.13
- net I_SENSE: now also U3.7; no longer U3.1
- net MISO: now also J8.3 (P3), U8.2 (MISO)
- net MOSI: no longer J8.5 (P5), U8.2 (MISO)
- net PWM: now also U1.1, U1.12; no longer U1.1, U1.12
- net SCLK: now also J8.5 (P5); no longer J8.3 (P3)
- net ~B: now also U1.8; no longer U1.6
- net ~D: now also U1.6; no longer U1.8
- net at R15.2, R18.1: now also U3.6 (-); no longer U3.2 (-)
- net at R16.2, R17.1: now also U3.5 (+); no longer U3.3 (+)
- new net: U1.10, U1.11, U1.9
- new net: U1.3, U1.4, U1.5
- no-connect marks 17 -> 16
Changed lines of the file:
@@
 Sheet 1 1
 Title "Zaza MK-1 48V Brushed DC motor controller"
-Date "2017-10-08"
-Rev "0"
+Date "2017-10-27"
+Rev "1"
 Comp "Alexandru Gagniuc"
 Comment1 ""
@@
 F 0 "QA1" H 5300 1550 50  0000 L CNN
 F 1 "DMN10" H 5300 1450 50  0000 L CNN
-F 2 "TO_SOT_Packages_SMD:SOT-404" H 5300 1600 50  0001 C CNN
+F 2 "TO-SMD:SOT-404-thermal-vias" H 5300 1600 50  0001 C CNN
 F 3 "" H 5100 1500 50  0001 C CNN
 	1    5100 1500
@@
 F 0 "QB1" H 5300 2150 50  0000 L CNN
 F 1 "DMN10" H 5300 2050 50  0000 L CNN
-F 2 "TO_SOT_Packages_SMD:SOT-404" H 5300 2200 50  0001 C CNN
+F 2 "TO-SMD:SOT-404-thermal-vias" H 5300 2200 50  0001 C CNN
 F 3 "" H 5100 2100 50  0001 C CNN
 	1    5100 2100
@@
 F 0 "QC1" H 6400 1550 50  0000 L CNN
 F 1 "DMN10" H 6400 1450 50  0000 L CNN
-F 2 "TO_SOT_Packages_SMD:SOT-404" H 6400 1600 50  0001 C CNN
+F 2 "TO-SMD:SOT-404-thermal-vias" H 6400 1600 50  0001 C CNN
 F 3 "" H 6200 1500 50  0001 C CNN
 	1    6200 1500
@@
 F 0 "QD1" H 6400 2150 50  0000 L CNN
 F 1 "DMN10" H 6400 2050 50  0000 L CNN
-F 2 "TO_SOT_Packages_SMD:SOT-404" H 6400 2200 50  0001 C CNN
+F 2 "TO-SMD:SOT-404-thermal-vias" H 6400 2200 50  0001 C CNN
 F 3 "" H 6200 2100 50  0001 C CNN
 	1    6200 2100
@@
 $Comp
 L LM358 U3
-U 1 1 59D68DCF
+U 2 1 59D68DCF
 P 9300 3200
 F 0 "U3" H 9300 3400 50  0000 L CNN
@@
 F 2 "Housings_SOIC:SOIC-8_3.9x4.9mm_Pitch1.27mm" H 9300 3200 50  0001 C CNN
 F 3 "" H 9300 3200 50  0001 C CNN
-	1    9300 3200
+	2    9300 3200
 	1    0    0    1
 $EndComp
@@
 $Comp
 L 74xx132 U1
-U 1 1 59D9916D
+U 4 1 59D9916D
 P 4900 3600
 F 0 "U1" H 4850 3650 50  0000 C CNN
@@
 F 2 "Housings_SOIC:SOIC-14_3.9x8.7mm_Pitch1.27mm" H 4800 3600 60  0001 C CNN
 F 3 "" H 4800 3600 60  0000 C CNN
-	1    4900 3600
+	4    4900 3600
 	-1   0    0    -1
 $EndComp
@@
 $Comp
 L 74xx132 U1
-U 4 1 59D9918C
+U 1 1 59D9918C
 P 6400 3600
 F 0 "U1" H 6350 3650 50  0000 C CNN
@@
 F 2 "Housings_SOIC:SOIC-14_3.9x8.7mm_Pitch1.27mm" H 6300 3600 60  0001 C CNN
 F 3 "" H 6300 3600 60  0000 C CNN
-	4    6400 3600
+	1    6400 3600
 	1    0    0    -1
 $EndComp
@@
 V
 $Comp
-L CONN_02X05 J3
-U 1 1 59DA4EF4
-P 5050 6800
-F 0 "J3" H 5050 7100 50  0000 C CNN
-F 1 "CONN_02X05" H 5050 6500 50  0000 C CNN
-F 2 "Connectors_Multicomp:Multicomp_MC9A12-1034_2x05x2.54mm_Straight" H 5050 5600 50  0001 C CNN
-F 3 "" H 5050 5600 50  0001 C CNN
-	1    5050 6800
-	-1   0    0    -1
-$EndComp
-$Comp
 L +48V #PWR06
 U 1 1 59DA5449
@@
 	1    1600 1000
 	1    0    0    -1
-$EndComp
-$Comp
-L GND #PWR08
-U 1 1 59DA6073
-P 5750 6900
-F 0 "#PWR08" H 5750 6650 50  0001 C CNN
-F 1 "GND" H 5750 6750 50  0000 C CNN
-F 2 "" H 5750 6900 50  0001 C CNN
-F 3 "" H 5750 6900 50  0001 C CNN
-	1    5750 6900
-	0    -1   1    0
 $EndComp
 $Comp
@@
 F 0 "D6" H 8300 6340 50  0000 C CNN
 F 1 "15.6V" H 8300 6160 50  0000 C CNN
-F 2 "Diodes_SMD:D_SOD-323" V 8300 6250 50  0001 C CNN
+F 2 "Diodes_SMD:D_SMA_Standard" V 8300 6250 50  0001 C CNN
 F 3 "" V 8300 6250 50  0001 C CNN
 	1    8300 6250
@@
 F 0 "D103" V 4100 1750 50  0000 C CNN
 F 1 "15.6V" V 4200 1625 50  0000 C CNN
-F 2 "Diodes_SMD:D_SOD-323" V 4300 1750 50  0001 C CNN
+F 2 "Diodes_SMD:D_SMA_Standard" V 4300 1750 50  0001 C CNN
 F 3 "" V 4300 1750 50  0001 C CNN
 	1    4300 1750
@@
 F 0 "D1" V 3300 6500 50  0000 L CNN
 F 1 "1N5711" V 3200 6300 50  0000 L CNN
-F 2 "Diodes_THT:D_DO-35_SOD27_P7.62mm_Horizontal" V 3200 6650 50  0001 C CNN
+F 2 "Diodes_SMD:D_MiniMELF_Standard" V 3200 6650 50  0001 C CNN
 F 3 "" V 3200 6650 50  0001 C CNN
 	1    3200 6650
@@
 $Comp
 L 74xx132 U1
-U 2 1 59EF5983
+U 3 1 59EF5983
 P 4000 3600
 F 0 "U1" H 3950 3650 50  0000 C CNN
@@
 F 2 "Housings_SOIC:SOIC-14_3.9x8.7mm_Pitch1.27mm" H 3900 3600 60  0001 C CNN
 F 3 "" H 3900 3600 60  0000 C CNN
-	2    4000 3600
+	3    4000 3600
 	-1   0    0    -1
 $EndComp
 $Comp
 L 74xx132 U1
-U 3 1 59EF6BC0
+U 2 1 59EF6BC0
 P 7300 3600
 F 0 "U1" H 7250 3650 50  0000 C CNN
@@
 F 2 "Housings_SOIC:SOIC-14_3.9x8.7mm_Pitch1.27mm" H 7200 3600 60  0001 C CNN
 F 3 "" H 7200 3600 60  0000 C CNN
-	3    7300 3600
+	2    7300 3600
 	1    0    0    -1
 $EndComp
@@
 F 0 "D203" V 6800 1725 50  0000 C CNN
 F 1 "15.6V" V 6900 1625 50  0000 C CNN
-F 2 "Diodes_SMD:D_SOD-323" V 7000 1750 50  0001 C CNN
+F 2 "Diodes_SMD:D_SMA_Standard" V 7000 1750 50  0001 C CNN
 F 3 "" V 7000 1750 50  0001 C CNN
 	1    7000 1750
@@
 	0    1    -1   0
 $EndComp
-Text Label 4800 7000 2    60   ~ 0
-CS_ADDR2
-Text Label 5300 7000 0    60   ~ 0
-CS_ADDR1
-Text Label 4800 6900 2    60   ~ 0
-CS_ADDR0
-Text Label 4800 6800 2    60   ~ 0
-SCLK
-Text Label 4800 6700 2    60   ~ 0
-MISO
-Text Label 4800 6600 2    60   ~ 0
-MOSI
 $Comp
 L R_Small R1
@@
 	1    0    0    -1
 $EndComp
-NoConn ~ 5300 6700
 Text Label 8400 4500 2    60   ~ 0
 SCLK
@@
 MOSI
 Text Label 6100 5000 3    60   ~ 0
-MOSI
+MISO
 Text Label 6000 5000 3    60   ~ 0
 ~CS_ROM
@@
 Text Label 1350 1800 0    60   ~ 0
 PWM
-Text Label 5300 6800 0    60   ~ 0
-PWM
-$Comp
-L +5V #PWR062
-U 1 1 59F3D397
-P 5300 6600
-F 0 "#PWR062" H 5300 6450 50  0001 C CNN
-F 1 "+5V" H 5300 6740 50  0000 C CNN
-F 2 "" H 5300 6600 50  0001 C CNN
-F 3 "" H 5300 6600 50  0001 C CNN
-	1    5300 6600
-	-1   0    0    -1
-$EndComp
 $Comp
 L GNDREF #PWR063
@@
 Entry Wire Line
 	4600 4900 4700 5000
+Text Label 4500 5000 3    60   ~ 0
+SCLK
 Text Label 4700 5000 3    60   ~ 0
-SCLK
+MISO
 Text Label 4600 5000 3    60   ~ 0
-MOSI
-Text Label 4500 5000 3    60   ~ 0
 MOSI
 Text Label 4400 5000 3    60   ~ 0
@@
 	6000 6400 6000 5000
 Wire Wire Line
-	5750 6900 5300 6900
-Wire Wire Line
 	1000 1900 2600 1900
 Wire Wire Line
@@
 F 0 "J200" H 800 2400 50  0000 C CNN
 F 1 "MX120G" V 900 1750 50  0000 C CNN
-F 2 "" H 800 1750 50  0001 C CNN
+F 2 "molex-120g:Molex_MX120G_02x06_3.5mm_36783-1201" H 800 1750 50  0001 C CNN
 F 3 "" H 800 1750 50  0001 C CNN
 	1    800  1750
