File: zaza-motor-controller.kicad_pcb (KiCad board)
At the start: 2 copper layers, 53 x 60 mm, 74 parts, among them J1 VIN, J2 VIN, J3 CONN_02X05, J4 CONN_02X01, J5 GS3, Q1 BC337, Q10 BC327, Q11 BC337, Q12 BC337, Q2 BC337, Q3 BC327, Q4 BC337, Q5 IXTA220, Q6 IXTA220, Q7 IXTA220, Q8 IXTA220, Q9 BC337, U1 74HC00, U2 74HC00, U3 LM358, U4 LM555N

Commit message: Rev1 dev
Parts:
- added C15: CP, Capacitors_THT:CP_Axial_L29.0mm_D20.0mm_P35.00mm_Horizontal, F.Cu at (83.0, 146.0)
- Q5, Q6, Q7, Q8, R9: moved to F.Cu
- moved D12 110.2 mm to (111.0, 185.0)
- moved Q10 110.2 mm to (114.0, 182.0)
- moved Q12 110.2 mm to (114.0, 186.0)
- moved Q9 110.2 mm to (114.0, 178.0)
- moved R11 110.2 mm to (109.0, 178.0)
- moved R12 110.2 mm to (109.0, 182.0)
- moved R13 110.2 mm to (109.0, 186.0)
- moved Q2 109.8 mm to (101.0, 178.1)
- moved D5 109.8 mm to (98.0, 185.0)
- moved Q1 109.8 mm to (101.0, 186.0)
- moved Q3 109.8 mm to (101.0, 182.0)
- moved R4 109.8 mm to (96.0, 186.0)
- moved R6 109.8 mm to (96.0, 178.0)
- moved R7 109.8 mm to (96.0, 182.0)
- moved J1 98.4 mm to (45.0, 143.0)
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Routing:
- net GND: track 293.1 -> 99.7 mm, vias 18 -> 9
- net +48V: track 137.1 -> 69.9 mm, vias 4 -> 36
- net VEE: track 52.1 -> 2.02 mm, vias 2 -> 0
- net +5V: track 77.7 -> 34.4 mm, vias 3 -> 0
- net /~C: track 43.1 -> 0.30 mm
- net /~A: track 41.0 -> 0.72 mm
- net /V_SENSE: track 37.5 -> 0.00 mm
- net /~D: track 35.9 -> 0.30 mm
- net HT: track 49.5 -> 15.8 mm
- net /~B: track 30.8 -> 0.75 mm
- net /I_SENSE: track 29.8 -> 4.97 mm
- net Net-(D10-Pad1): track 13.2 -> 36.8 mm, vias 1 -> 0
- net /PUMP_OSC: track 34.0 -> 14.3 mm
- net /M+: track 43.4 -> 24.8 mm, vias 0 -> 18
- net GNDPWR: track 29.9 -> 14.1 mm
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- added copper zone on F.Cu, net GNDPWR
- added copper zone on F.Cu, net Net-(Q6-Pad3)
Other:
- board size 53 x 60 mm -> 108 x 57.5 mm
- board text removed: "Designed by Alexandru Gagniuc"
- board text removed: "MAX"

Commit message: Layout choochiness over nine thousand
Parts:
- removed C10, C4, C5: 1uF, Capacitors_SMD:C_0805
- removed D10, D11, D12: BAT5H17, Diodes_SMD:D_MiniMELF_Standard
- removed D2: BAR43, TO_SOT_Packages_SMD:SOT-23
- removed Q10, Q3: BC327, TO_SOT_Packages_SMD:SOT-23
- removed Q11, Q12, Q2, Q4, Q9: BC337, TO_SOT_Packages_SMD:SOT-23
- removed Q5, Q6, Q7, Q8: IXTA220, TO_SOT_Packages_SMD:SOT-404
- removed R21: 180k, Resistors_SMD:R_0805
- removed R22, R23: 3.3k, Resistors_SMD:R_0805
- removed TP2: -8V, Measurement_Points:Test_Point_Keystone_5000-5004_Miniature
- removed TP3: 56V, Measurement_Points:Test_Point_Keystone_5000-5004_Miniature
- removed U2: 74HC00, Housings_SOIC:SOIC-14_3.9x8.7mm_Pitch1.27mm
- added C100: 220n, Capacitors_SMD:C_0805, F.Cu at (176.0, 103.0)
- added C200: 220n, Capacitors_SMD:C_0805, F.Cu at (189.0, 103.0)
- added D100: 1N..., Diodes_SMD:D_MiniMELF_Standard, F.Cu at (166.0, 102.5)
- added D101: 1N..., Diodes_SMD:D_MiniMELF_Standard, F.Cu at (166.0, 98.0)
- added D102: 1N..., Diodes_SMD:D_MiniMELF_Standard, F.Cu at (166.0, 100.2)
- added D200: 1N..., Diodes_SMD:D_MiniMELF_Standard, F.Cu at (183.0, 100.0)
- added D201: 1N..., Diodes_SMD:D_MiniMELF_Standard, F.Cu at (189.0, 97.8)
- added D202: 1N..., Diodes_SMD:D_MiniMELF_Standard, F.Cu at (189.0, 100.0)
- added F1: 100mA, Resistors_SMD:R_1206, F.Cu at (153.0, 70.0)
- added J200: MX120G, molex-120g:Molex_MX120G_02x06_3.5mm_36783-1201, F.Cu at (112.5, 80.0)
- added J6: V, Pin_Headers:Pin_Header_Straight_2x01_Pitch2.54mm, F.Cu at (138.0, 99.0)
- added J7: CAL_EN, Pin_Headers:Pin_Header_Straight_2x01_Pitch2.54mm, F.Cu at (232.0, 115.5)
- added J8: CONN_01X06, Pin_Headers:Pin_Header_Straight_1x06_Pitch2.54mm, F.Cu at (150.0, 159.8)
- added QA1: DMN10, TO-SMD:SOT-404-thermal-vias, F.Cu at (172.6, 73.0)
- added QB1: DMN10, TO-SMD:SOT-404-thermal-vias, F.Cu at (191.6, 73.0)
- added QC1: DMN10, TO-SMD:SOT-404-thermal-vias, F.Cu at (172.6, 87.0)
- added QD1: DMN10, TO-SMD:SOT-404-thermal-vias, F.Cu at (191.6, 87.0)
- added R100: 10k, Resistors_SMD:R_0805, F.Cu at (161.0, 97.0)
- added R101: 10k, Resistors_SMD:R_0805, F.Cu at (162.1, 99.0)
- added R102: 1k, Resistors_SMD:R_0805, F.Cu at (171.0, 97.0)
- added R103: 0R, Resistors_SMD:R_0805, F.Cu at (173.0, 97.0)
- added R104: 1k, Resistors_SMD:R_0805, F.Cu at (175.0, 97.0)
- added R200: 10k, Resistors_SMD:R_0805, F.Cu at (193.9, 97.8)
- added R201: 10k, Resistors_SMD:R_0805, F.Cu at (194.1, 101.0)
- added R202: 1k, Resistors_SMD:R_0805, F.Cu at (194.1, 103.0)
- added R203: 0R, Resistors_SMD:R_0805, F.Cu at (194.1, 105.0)
- added R204: 1k, Resistors_SMD:R_0805, F.Cu at (194.0, 107.0)
- added SCD-80: D_SCD80, Diodes_SMD:D_SCD80, F.Cu at (45.0, 28.0)
- added SOD-323: D_SOD-323, Diodes_SMD:D_SOD-323, F.Cu at (38.0, 28.0)
- added SOD-523: D_SOD-523, Diodes_SMD:D_SOD-523, F.Cu at (42.0, 28.0)
- added U10: LM7805CT, TO_SOT_Packages_SMD:SOT-223-3Lead_TabPin2, F.Cu at (72.0, 69.0)
- added U100: IRS2003, Housings_SOIC:SOIC-8_3.9x4.9mm_Pitch1.27mm, F.Cu at (172.0, 103.0)
- added U200: IRS2003, Housings_SOIC:SOIC-8_3.9x4.9mm_Pitch1.27mm, F.Cu at (184.0, 104.0)
- added U5: 74xx138, Housings_SOIC:SOIC-16_3.9x9.9mm_Pitch1.27mm, F.Cu at (136.0, 91.0)
- added U6: 74xx595, Housings_SOIC:SOIC-16_3.9x9.9mm_Pitch1.27mm, F.Cu at (145.0, 91.0)
- added U8: AT25XX, Housings_SOIC:SOIC-8_3.9x4.9mm_Pitch1.27mm, F.Cu at (238.0, 116.6)
- added U9: ADS1018, Housings_SSOP:MSOP-10_3x3mm_Pitch0.5mm, F.Cu at (19.0, 89.0)
- added sod-123f: D_SOD-123F, Diodes_SMD:D_SOD-123F, F.Cu at (34.0, 28.0)
- added sod123: D_SOD-123, Diodes_SMD:D_SOD-123, F.Cu at (30.0, 28.0)
- C1: value 100p -> 1n
- C15: value CP -> 100u 100V; footprint Capacitors_THT:CP_Axial_L29.0mm_D20.0mm_P35.00mm_Horizontal -> Capacitors_THT:CP_Axial_L29.0mm_D16.0mm_P35.00mm_Horizontal
- C2: value 1nF -> 100p
- D4, D6: value BAR43 -> 15.6V; footprint TO_SOT_Packages_SMD:SOT-23 -> Diodes_SMD:D_SOD-323
- D5: value BAT5H17 -> 15.6V; footprint Diodes_SMD:D_MiniMELF_Standard -> Diodes_SMD:D_SOD-323
- J3: footprint Connectors:IDC_Header_Straight_10pins -> Connectors_Multicomp:Multicomp_MC9A12-1034_2x05x2.54mm_Straight
- J5: value GS3 -> U; footprint Connectors:GS3 -> Pin_Headers:Pin_Header_Straight_2x01_Pitch2.54mm
- Q1: value BC337 -> NZT605; footprint TO_SOT_Packages_SMD:SOT-23 -> TO_SOT_Packages_SMD:SOT-223-3Lead_TabPin2
- R11, R13: value 10k -> 50R; footprint Resistors_SMD:R_0805 -> Resistors_SMD:R_2010
- R12: value 50k -> 10k
- R14: value 10k -> 180k
- R2: value 10k -> 0R
- R3: value 47k -> 10k
- R4: value 10k -> 47k
- R5, R6, R8: value 10k -> 1M
- R7: value 50k -> 1M
- TP1: value ~PWM -> 60V
- TP4: value ~A -> A
- TP7: value ~C -> C
- moved R6 141.4 mm to (197.0, 79.0), turned to 0 degrees
- moved R7 127.6 mm to (197.0, 104.0)
- moved D5 124.0 mm to (191.0, 103.0)
- moved R13 123.7 mm to (66.0, 70.0), turned to 90 degrees
- moved J2 121.8 mm to (120.0, 54.0)
- moved Q1 121.1 mm to (147.0, 74.0)
- moved R9 118.9 mm to (183.0, 60.0)
- moved D4 117.3 mm to (178.0, 103.0), turned to 90 degrees
- moved R11 112.0 mm to (153.0, 75.0)
- moved J1 111.4 mm to (112.0, 54.0)
- moved R10 110.8 mm to (233.0, 121.0), turned to 0 degrees
- moved R12 109.6 mm to (149.0, 80.0), turned to 0 degrees
- moved R8 109.2 mm to (199.0, 95.0), turned to 180 degrees
- moved U1 109.2 mm to (145.0, 103.0), turned to 0 degrees
- moved C8 105.9 mm to (70.0, 75.0), turned to 0 degrees
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Connections:
- C1 pad 2: GND -> GNDPWR
- C2 pad 2: GND -> GNDPWR
- C6 pad 1: Net-(C10-Pad2) -> HT
- C6 pad 2: GND -> +48V
- C7 pad 2: Net-(C3-Pad1) -> GNDPWR
- C8 pad 2: Net-(C4-Pad1) -> GND
- C9 pad 1: HT -> +5V
- C9 pad 2: Net-(C5-Pad1) -> GND
- D3 pad 2: Net-(C7-Pad1) -> (no net)
- D3 pad 3: Net-(C5-Pad1) -> HT
- D4 pad 1: VEE -> Net-(C100-Pad1)
- D4 pad 2: Net-(C10-Pad2) -> Net-(C100-Pad2)
- D5 pad 1: Net-(D5-Pad1) -> Net-(C200-Pad1)
- D5 pad 2: Net-(D5-Pad2) -> Net-(C200-Pad2)
- D6 pad 2: Net-(D6-Pad2) -> GNDPWR
- J3 pad 10: /I_SENSE -> /CS_ADDR2
- J3 pad 2: /U -> /MOSI
- J3 pad 3: GND -> (no net)
- J3 pad 4: /V -> /MISO
- J3 pad 5: GND -> /PWM
- J3 pad 6: /EN -> /SCLK
- J3 pad 8: /V_SENSE -> /CS_ADDR0
- J3 pad 9: GND -> /CS_ADDR1
- J5 pad 1: GND -> /A
- Q1 pad 1: Net-(D5-Pad2) -> Net-(C7-Pad1)
- Q1 pad 2: GND -> Net-(Q1-Pad2)
- Q1 pad 3: Net-(D5-Pad1) -> +15V
- R1 pad 1: GND -> GNDREF
- R1 pad 2: GNDPWR -> GND
- R10 pad 1: +48V -> Net-(J7-Pad2)
- R10 pad 2: Net-(D11-Pad1) -> GND
- R11 pad 1: HT -> Net-(F1-Pad1)
- R11 pad 2: Net-(Q10-Pad1) -> Net-(Q1-Pad2)
- R12 pad 1: Net-(Q10-Pad1) -> Net-(C7-Pad1)
- R12 pad 2: Net-(D12-Pad1) -> Net-(Q1-Pad2)
- R13 pad 1: /~C -> +15V
- R13 pad 2: Net-(D12-Pad2) -> Net-(C8-Pad1)
- R14 pad 1: /~D -> /V_SENSE
- R14 pad 2: Net-(D11-Pad2) -> +48V
- R16 pad 1: Net-(Q6-Pad3) -> Net-(QB1-Pad3)
- R2 pad 1: +5V -> GND
- R2 pad 2: Net-(R2-Pad2) -> GNDPWR
- R3 pad 1: Net-(R2-Pad2) -> +15V
- R3 pad 2: Net-(C2-Pad1) -> Net-(R3-Pad2)
- R4 pad 1: /~A -> Net-(R3-Pad2)
- R4 pad 2: Net-(D5-Pad2) -> Net-(C2-Pad1)
- R5 pad 1: /~B -> Net-(QA1-Pad1)
- R5 pad 2: Net-(D10-Pad2) -> /M+
- R6 pad 1: HT -> Net-(QB1-Pad1)
- R6 pad 2: Net-(Q2-Pad1) -> Net-(QB1-Pad3)
- R7 pad 1: Net-(Q2-Pad1) -> Net-(QC1-Pad1)
- R7 pad 2: Net-(D5-Pad1) -> /M-
- R8 pad 1: +48V -> Net-(QD1-Pad1)
- R8 pad 2: Net-(D10-Pad1) -> Net-(QB1-Pad3)
- R9 pad 1: Net-(Q6-Pad3) -> Net-(QB1-Pad3)
- TP1 pad 1: /~PWM -> HT
- TP4 pad 1: /~A -> /A
- TP7 pad 1: /~C -> /C
- U1 pad 1: /EN -> /PWM
- U1 pad 10: /~V -> Net-(U1-Pad10)
- U1 pad 11: /~V -> Net-(U1-Pad10)
- U1 pad 12: /V -> /PWM
- U1 pad 13: /V -> /C
- U1 pad 2: /EN -> /A
- U1 pad 3: /~PWM -> Net-(U1-Pad3)
- U1 pad 4: /V -> Net-(U1-Pad3)
- U1 pad 5: /~PWM -> Net-(U1-Pad3)
- U1 pad 6: /~D -> /~B
- U1 pad 8: /~C -> /~D
- U1 pad 9: /~PWM -> Net-(U1-Pad10)
- U3 pad 4: +5V -> GND
- U3 pad 8: Net-(J5-Pad2) -> +5V
- U4 pad 1: GND -> GNDPWR
- U4 pad 4: +5V -> +15V
- U4 pad 7: Net-(R2-Pad2) -> Net-(R3-Pad2)
- U4 pad 8: +5V -> +15V
Routing:
- net GNDPWR: track 14.1 -> 125.0 mm, vias 0 -> 2
- net GND: track 99.7 -> 28.4 mm, vias 9 -> 1
- net +48V: track 69.9 -> 134.4 mm, vias 36 -> 0
- net /CS_ADDR0: track 0.00 -> 47.2 mm
- net /CS_ADDR2: track 0.00 -> 42.5 mm
- net Net-(QB1-Pad1): track 0.00 -> 40.2 mm, vias 0 -> 2
- net /CS_ADDR1: track 0.00 -> 38.8 mm
- net /C: track 0.00 -> 38.1 mm
- net Net-(D10-Pad1): track 36.8 -> 0.00 mm
- net /M+: track 24.8 -> 60.2 mm, vias 18 -> 2
- net /~D: track 0.30 -> 35.3 mm
- net Net-(QC1-Pad1): track 0.00 -> 31.0 mm
- net /M-: track 24.8 -> 55.7 mm, vias 18 -> 0
- net +5V: track 34.4 -> 3.88 mm
- net /MOSI: track 0.00 -> 28.2 mm
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- added copper zone on F.Cu, net +48V
- added copper zone on B.Cu, net GNDPWR
- added copper zone on F.Cu, net Net-(QB1-Pad3)
- removed copper zone on B.Cu, net +48V
- removed copper zone on F.Cu, net Net-(Q6-Pad3)
Other:
- outline, holes or cut-outs redrawn
- board text added: "5V"
- board text added: "GND"
- board text added: "MISO"
- board text added: "MOSI"
- board text added: "NC"
- board text added: "SCLK"
- board text added: "~CSA0"
- board text added: "~CSA1"
- board text added: "~CSA2"
- board text removed: "Amp"
- board text removed: "U"
- board text removed: "V"
- board text removed: "Volt"

Commit message: moar layout
Parts:
- removed D4, D5: 15.6V, Diodes_SMD:D_SOD-323
- removed J3: CONN_02X05, Connectors_Multicomp:Multicomp_MC9A12-1034_2x05x2.54mm_Straight
- removed SCD-80: D_SCD80, Diodes_SMD:D_SCD80
- removed SOD-323: D_SOD-323, Diodes_SMD:D_SOD-323
- removed SOD-523: D_SOD-523, Diodes_SMD:D_SOD-523
- removed sod-123f: D_SOD-123F, Diodes_SMD:D_SOD-123F
- removed sod123: D_SOD-123, Diodes_SMD:D_SOD-123
- added D103: 15.6V, Diodes_SMD:D_SMA_Standard, F.Cu at (158.0, 91.5)
- added D203: 15.6V, Diodes_SMD:D_SMA_Standard, F.Cu at (151.5, 100.5)
- D1: footprint Diodes_THT:D_DO-35_SOD27_P7.62mm_Horizontal -> Diodes_SMD:D_MiniMELF_Standard
- D6: footprint Diodes_SMD:D_SOD-323 -> Diodes_SMD:D_SMA_Standard
- moved R3 130.6 mm to (159.0, 54.0), turned to 270 degrees
- moved C2 128.4 mm to (161.0, 58.0)
- moved U4 128.4 mm to (154.0, 56.0), turned to 0 degrees
- moved C1 128.4 mm to (159.0, 58.0), turned to 270 degrees
- moved R4 128.2 mm to (162.0, 55.0), turned to 0 degrees
- moved J7 117.5 mm to (115.0, 104.0), turned to 180 degrees
- moved R15 114.4 mm to (138.0, 72.0)
- moved R18 112.7 mm to (136.0, 72.0), turned to 90 degrees
- moved D1 111.8 mm to (160.0, 72.0)
- moved C3 109.6 mm to (164.0, 73.0), turned to 90 degrees
- moved C6 108.5 mm to (164.0, 76.0), turned to 0 degrees
- moved R17 107.8 mm to (133.0, 77.0), turned to 270 degrees
- moved R19 107.7 mm to (131.0, 77.0)
- moved R10 107.0 mm to (127.0, 106.0), turned to 270 degrees
- moved U8 106.7 mm to (132.0, 104.5)
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Connections:
- J8 pad 3: /SCLK -> /MISO
- J8 pad 5: /MOSI -> /SCLK
- U1 pad 13: /C -> /A
- U1 pad 2: /A -> /C
- U1 pad 6: /~B -> /~D
- U1 pad 8: /~D -> /~B
- U3 pad 1: /I_SENSE -> (no net)
- U3 pad 2: Net-(R15-Pad2) -> (no net)
- U3 pad 3: Net-(R16-Pad2) -> (no net)
- U3 pad 5: (no net) -> Net-(R16-Pad2)
- U3 pad 6: (no net) -> Net-(R15-Pad2)
- U3 pad 7: (no net) -> /I_SENSE
- U8 pad 2: /MOSI -> /MISO
Routing:
- net +15V: track 3.97 -> 173.9 mm, vias 0 -> 3
- net GND: track 28.4 -> 142.0 mm, vias 1 -> 14
- net +5V: track 3.88 -> 113.6 mm, vias 0 -> 7
- net Net-(QB1-Pad3): track 19.6 -> 90.0 mm, vias 0 -> 26
- net +48V: track 134.4 -> 193.8 mm, vias 0 -> 3
- net /V_SENSE: track 0.00 -> 56.6 mm
- net GNDPWR: track 125.0 -> 172.1 mm, vias 2 -> 6
- net /A: track 0.00 -> 45.8 mm, vias 0 -> 1
- net /~B: track 0.75 -> 44.0 mm, vias 0 -> 1
- net /PUMP_OSC: track 0.95 -> 40.7 mm, vias 0 -> 2
- net Net-(D202-Pad2): track 2.94 -> 39.7 mm
- net Net-(D201-Pad2): track 2.37 -> 37.0 mm
- net Net-(D102-Pad2): track 0.00 -> 34.5 mm, vias 0 -> 2
- net /MOSI: track 28.2 -> 59.1 mm, vias 0 -> 3
- net /SCLK: track 26.4 -> 56.4 mm, vias 0 -> 2
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- added copper zone on B.Cu, net +48V
- added copper zone on B.Cu, net Net-(QB1-Pad3)
- removed copper zone on F.Cu, net +48V
Other:
- outline, holes or cut-outs redrawn
- net class Default: via_drill 0.4 -> 0.3
- net class PWR: via_drill 0.4 -> 0.3
- net class PWR-small: via_drill 0.4 -> 0.3
- board text added: "Designed by Hugh E. Dick"
- board text added: "~DAC"
- board text removed: "NC"
- board text removed: "PWM"
- board text removed: "~CSA0"
- board text removed: "~CSA1"
- board text removed: "~CSA2"

Commit message: fix the darn author's name
Other:
- board text added: "Designed by Alexandru Gagniuc"
- board text removed: "Designed by Hugh E. Dick"
Changed lines of the file:
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@@
   (title_block
     (title "Zaza MK-1 48V Brushed DC motor controller")
-    (date 2017-10-08)
-    (rev 0)
+    (date 2017-10-27)
+    (rev 1)
     (company "Alexandru Gagniuc")
   )
@@
     )
   )
-  (gr_text "Designed by Hugh E. Dick" (at 142.5 62) (layer F.SilkS)
+  (gr_text "Designed by Alexandru Gagniuc" (at 144 62) (layer F.SilkS)
     (effects (font (size 1.5 1.5) (thickness 0.3)))
   )
